File: connectors.kicad_sch (KiCad schematic)
At the start: 4 parts, among them J1 Conn_01x04_Male, J2 Conn_01x09_Male, J3 Conn_01x04_Male, J4 Conn_02x03_Odd_Even

Commit message: Completed the symbol foot prints
Parts:
- J1, J2, J3: footprint (none) -> Connector_PinHeader_2.54mm:PinHeader_1x01_P2.54mm_Vertical
- J4: footprint (none) -> Connector_PinHeader_2.54mm:PinHeader_2x03_P2.54mm_Vertical
Changed lines of the file:
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@@
     (property "Reference" "J3" (id 0) (at 107.315 53.34 0))
     (property "Value" "Conn_01x04_Male" (id 1) (at 107.315 55.88 0))
-    (property "Footprint" "" (id 2) (at 106.68 60.96 0)
+    (property "Footprint" "Connector_PinHeader_2.54mm:PinHeader_1x01_P2.54mm_Vertical" (id 2) (at 106.68 60.96 0)
       (effects (font (size 1.27 1.27)) hide)
     )
@@
     (property "Reference" "J2" (id 0) (at 75.565 76.2 0))
     (property "Value" "Conn_01x09_Male" (id 1) (at 75.565 78.74 0))
-    (property "Footprint" "" (id 2) (at 74.93 91.44 0)
+    (property "Footprint" "Connector_PinHeader_2.54mm:PinHeader_1x01_P2.54mm_Vertical" (id 2) (at 74.93 91.44 0)
       (effects (font (size 1.27 1.27)) hide)
     )
@@
     (property "Reference" "J1" (id 0) (at 74.295 57.15 0))
     (property "Value" "Conn_01x04_Male" (id 1) (at 74.295 59.69 0))
-    (property "Footprint" "" (id 2) (at 73.66 64.77 0)
+    (property "Footprint" "Connector_PinHeader_2.54mm:PinHeader_1x01_P2.54mm_Vertical" (id 2) (at 73.66 64.77 0)
       (effects (font (size 1.27 1.27)) hide)
     )
@@
     (property "Reference" "J4" (id 0) (at 110.49 80.01 0))
     (property "Value" "Conn_02x03_Odd_Even" (id 1) (at 110.49 82.55 0))
-    (property "Footprint" "" (id 2) (at 109.22 88.9 0)
+    (property "Footprint" "Connector_PinHeader_2.54mm:PinHeader_2x03_P2.54mm_Vertical" (id 2) (at 109.22 88.9 0)
       (effects (font (size 1.27 1.27)) hide)
     )

Commit message: Finished wiring
Connections:
- net GND: now reaches J3.1 (Pin_1)
- net GND: now also J1.1 (Pin_1), J2.8 (Pin_8), J4.6 (Pin_6)
- net Vcc: now reaches J3.2 (Pin_2)
- net Vcc: now also J1.2 (Pin_2), J2.9 (Pin_9), J4.2 (Pin_2)
- net RX: now reaches J3.3 (Pin_3)
- net TX: now reaches J3.4 (Pin_4)
- net D2: now reaches J2.1 (Pin_1)
- net D3: now reaches J2.2 (Pin_2)
- net D4: now reaches J2.3 (Pin_3)
- net D5: now reaches J2.4 (Pin_4)
- net D6: now reaches J2.5 (Pin_5)
- net D7: now reaches J2.6 (Pin_6)
- net D8: now reaches J2.7 (Pin_7)
- net SDA: now reaches J1.3 (Pin_3)
- net SCK: now reaches J1.4 (Pin_4)
- net SCK: now also J4.3 (Pin_3)
- net MISO: now reaches J4.1 (Pin_1)
- net MOSI: now reaches J4.4 (Pin_4)
- net RESET: now reaches J4.5 (Pin_5)
Changed lines of the file:
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@@
 (kicad_sch (version 20211123) (generator eeschema)
   (paper "A4")
+  (hierarchical_label "D6" (shape bidirectional) (at 80.01 91.44 0)
+    (effects (font (size 1.27 1.27)) (justify left))
+  )
+  (hierarchical_label "D2" (shape bidirectional) (at 80.01 81.28 0)
+    (effects (font (size 1.27 1.27)) (justify left))
+  )
+  (hierarchical_label "GND" (shape passive) (at 116.84 91.44 0)
+    (effects (font (size 1.27 1.27)) (justify left))
+  )
+  (hierarchical_label "D8" (shape bidirectional) (at 80.01 96.52 0)
+    (effects (font (size 1.27 1.27)) (justify left))
+  )
+  (hierarchical_label "GND" (shape passive) (at 80.01 99.06 0)
+    (effects (font (size 1.27 1.27)) (justify left))
+  )
+  (hierarchical_label "Vcc" (shape passive) (at 78.74 64.77 0)
+    (effects (font (size 1.27 1.27)) (justify left))
+  )
+  (hierarchical_label "GND" (shape passive) (at 78.74 62.23 0)
+    (effects (font (size 1.27 1.27)) (justify left))
+  )
+  (hierarchical_label "D5" (shape bidirectional) (at 80.01 88.9 0)
+    (effects (font (size 1.27 1.27)) (justify left))
+  )
+  (hierarchical_label "Vcc" (shape passive) (at 111.76 60.96 0)
+    (effects (font (size 1.27 1.27)) (justify left))
+  )
+  (hierarchical_label "SDA" (shape bidirectional) (at 78.74 67.31 0)
+    (effects (font (size 1.27 1.27)) (justify left))
+  )
+  (hierarchical_label "D3" (shape bidirectional) (at 80.01 83.82 0)
+    (effects (font (size 1.27 1.27)) (justify left))
+  )
+  (hierarchical_label "RX" (shape input) (at 111.76 63.5 0)
+    (effects (font (size 1.27 1.27)) (justify left))
+  )
+  (hierarchical_label "SCK" (shape passive) (at 104.14 88.9 180)
+    (effects (font (size 1.27 1.27)) (justify right))
+  )
+  (hierarchical_label "Vcc" (shape passive) (at 80.01 101.6 0)
+    (effects (font (size 1.27 1.27)) (justify left))
+  )
+  (hierarchical_label "TX" (shape output) (at 111.76 66.04 0)
+    (effects (font (size 1.27 1.27)) (justify left))
+  )
+  (hierarchical_label "MOSI" (shape input) (at 116.84 88.9 0)
+    (effects (font (size 1.27 1.27)) (justify left))
+  )
+  (hierarchical_label "SCK" (shape bidirectional) (at 78.74 69.85 0)
+    (effects (font (size 1.27 1.27)) (justify left))
+  )
+  (hierarchical_label "RESET" (shape passive) (at 104.14 91.44 180)
+    (effects (font (size 1.27 1.27)) (justify right))
+  )
+  (hierarchical_label "Vcc" (shape passive) (at 116.84 86.36 0)
+    (effects (font (size 1.27 1.27)) (justify left))
+  )
+  (hierarchical_label "GND" (shape passive) (at 111.76 58.42 0)
+    (effects (font (size 1.27 1.27)) (justify left))
+  )
+  (hierarchical_label "D4" (shape bidirectional) (at 80.01 86.36 0)
+    (effects (font (size 1.27 1.27)) (justify left))
+  )
+  (hierarchical_label "D7" (shape bidirectional) (at 80.01 93.98 0)
+    (effects (font (size 1.27 1.27)) (justify left))
+  )
+  (hierarchical_label "MISO" (shape output) (at 104.14 86.36 180)
+    (effects (font (size 1.27 1.27)) (justify right))
+  )
   (symbol (lib_id "Connector:Conn_01x04_Male") (at 106.68 60.96 0) (unit 1)
     (in_bom yes) (on_board yes)
@@
       (effects (font (size 1.27 1.27)) hide)
     )
-    (property "Purpose" "ICSP" (id 4) (at 97.79 91.44 0))
+    (property "Purpose" "ICSP" (id 4) (at 110.49 95.25 0))
     (pin "1")
     (pin "2")
